Commit message: URDF numbers

File: urdf/robot.urdf.xacro (robot description, xacro)
@@ -1,4 +1,4 @@
 <?xml version="1.0" ?>
-<robot name="makerspet_loki" xmlns:xacro="http://ros.org/wiki/xacro">
+<robot name="makerspet_mini" xmlns:xacro="http://ros.org/wiki/xacro">
   <!-- https://classic.gazebosim.org/tutorials?tut=ros_gzplugins&cat=connect_ros -->
   <!-- https://classic.gazebosim.org/tutorials?tut=ros_urdf&cat=connect_ros -->
@@ -7,12 +7,12 @@
   <!-- ****************** ROBOT DIMENSIONS ****************** -->
   <!-- Units: meters, degrees, kg, N*m, m/s2 -->
-  <xacro:property name="wheel_diameter" value="0.067"/>
-  <xacro:property name="wheel_width" value="0.029"/>
-  <xacro:property name="caster_diameter" value="0.04"/>
+  <xacro:property name="wheel_diameter" value="0.043"/>
+  <xacro:property name="wheel_width" value="0.005"/>
+  <xacro:property name="caster_diameter" value="0.017"/>
   <!-- Caster center to base edge -->
   <xacro:property name="caster_inset" value="0.0386"/>
-  <xacro:property name="floor_clearance" value="0.018"/>
-  <xacro:property name="base_diameter" value="0.2042"/>
-  <xacro:property name="wheel_base" value="0.159063"/>
+  <xacro:property name="floor_clearance" value="0.0149"/>
+  <xacro:property name="base_diameter" value="0.124"/>
+  <xacro:property name="wheel_base" value="0.104243"/>
   <xacro:property name="lower_cylinder_height" value="0.1227"/>
   <xacro:property name="lower_to_upper_cylinders_gap" value="0.0195"/>
@@ -36,6 +36,7 @@
   <xacro:property name="imu_joint_dz" value="0"/>
   <!-- imu_joint_rpy: [0.0, 0.0, 0.0] -->
-  <xacro:property name="motor_stall_torque" value="0.49"/>
-  <xacro:property name="max_wheel_acceleration" value="5"/>
+  <!-- N*m -->
+  <xacro:property name="motor_stall_torque" value="0.171616375"/>
+  <xacro:property name="max_wheel_acceleration" value="1"/>
   <xacro:property name="lower_cylinder_mass" value="0.500"/>
   <!-- caster and battery weight -->
@@ -282,5 +283,5 @@
       <origin xyz="0 0 0" rpy="0 0 0"/>
       <geometry>
-        <mesh filename="package://makerspet_loki/mesh/head.stl" scale="${0.001*base_diameter} ${0.001*base_diameter} ${0.001*head_height*2}"/>
+        <mesh filename="package://makerspet_mini/mesh/head.stl" scale="${0.001*base_diameter} ${0.001*base_diameter} ${0.001*head_height*2}"/>
       </geometry>
       <material name="red"/>

Commit message: Track tweak

File: urdf/robot.urdf.xacro (robot description, xacro)
@@ -8,5 +8,5 @@
   <!-- Units: meters, degrees, kg, N*m, m/s2 -->
   <xacro:property name="wheel_diameter" value="0.043"/>
-  <xacro:property name="wheel_width" value="0.005"/>
+  <xacro:property name="wheel_width" value="0.0055"/>
   <xacro:property name="caster_diameter" value="0.017"/>
   <!-- Caster center to base edge -->
@@ -14,5 +14,5 @@
   <xacro:property name="floor_clearance" value="0.0149"/>
   <xacro:property name="base_diameter" value="0.124"/>
-  <xacro:property name="wheel_base" value="0.104243"/>
+  <xacro:property name="wheel_base" value="0.105043"/>
   <xacro:property name="lower_cylinder_height" value="0.1227"/>
   <xacro:property name="lower_to_upper_cylinders_gap" value="0.0195"/>

Commit message: Cleanup

File: urdf/robot.urdf.xacro (robot description, xacro)
@@ -21,19 +21,4 @@
   <xacro:property name="upper_cylinder_height" value="0.003"/>
   <xacro:property name="head_height" value="0.09"/>
-  <xacro:property name="tablet_width" value="0.1669"/>
-  <xacro:property name="tablet_height" value="0.0781"/>
-  <xacro:property name="tablet_thickness" value="0.009"/>
-  <!-- Zero - tablet faces straight forward -->
-  <xacro:property name="tablet_pitch_angle" value="20"/>
-  <!-- Upper cylinder's front to tablet bottom's center -->
-  <xacro:property name="tablet_inset" value="0.07"/>
-  <xacro:property name="color_camera_diameter" value="0.004"/>
-  <!-- Tablet edge to camera center -->
-  <xacro:property name="color_camera_inset" value="0.008"/>
-  <!-- Delta xyz from tablet center -->
-  <xacro:property name="imu_joint_dx" value="0"/>
-  <xacro:property name="imu_joint_dy" value="0"/>
-  <xacro:property name="imu_joint_dz" value="0"/>
-  <!-- imu_joint_rpy: [0.0, 0.0, 0.0] -->
   <!-- N*m -->
   <xacro:property name="motor_stall_torque" value="0.171616375"/>
@@ -46,11 +31,6 @@
   <xacro:property name="upper_cylinder_mass" value="0.100"/>
   <xacro:property name="head_mass" value="0.200"/>
-  <xacro:property name="tablet_mass" value="0.200"/>
   <!-- ****************** **************** ****************** -->
   <xacro:property name="DEG2RAD" value="0.0174533"/>
-  <xacro:property name="color_camera_thickness" value="0.0001"/>
-  <xacro:property name="imu_xlen" value="0.001"/>
-  <xacro:property name="imu_ylen" value="0.002"/>
-  <xacro:property name="imu_zlen" value="0.004"/>
   <material name="black">
       <color rgba="0 0 0 1.0"/>
@@ -295,87 +275,4 @@
     <xacro:solid_semi_ellipsoid_inertia m="${head_mass}" x="${base_diameter/2}" y="${base_diameter/2}" z="${head_height}"/>
   </link>
-  <joint name="tablet_joint" type="fixed">
-    <parent link="head_link"/>
-    <child link="tablet_link"/>
-    <origin xyz="${base_diameter/2 - tablet_inset} 0 0" rpy="0 ${-tablet_pitch_angle*DEG2RAD} 0"/>
-  </joint>
-  <link name="tablet_link">
-    <visual>
-      <origin xyz="0 0 ${tablet_height/2}" rpy="${pi/2} 0 ${pi/2}"/>
-      <geometry>
-        <box size="${tablet_width} ${tablet_height} ${tablet_thickness}"/>
-      </geometry>
-      <material name="light_black"/>
-    </visual>
-   <collision>
-      <origin xyz="0 0 ${tablet_height/2}" rpy="${pi/2} 0 ${pi/2}"/>
-      <origin xyz="0 0 0.03905" rpy="${pi/2} 0 ${pi/2}"/>
-      <geometry>
-        <box size="${tablet_width} ${tablet_height} ${tablet_thickness}"/>
-      </geometry>
-    </collision>
-    <xacro:solid_box_inertia m="${tablet_mass}" x="${tablet_width}" y="${tablet_height}" z="${tablet_thickness}"/>
-  </link>
-  <joint name="color_camera_joint" type="fixed">
-    <parent link="tablet_link"/>
-    <child link="color_camera_link"/>
-    <origin xyz="${tablet_thickness/2-color_camera_thickness} ${color_camera_inset - tablet_width/2} ${tablet_height/2}" rpy="0 0 0"/>
-  </joint>
-  <link name="color_camera_link">
-    <visual>
-      <origin xyz="0 0 0" rpy="0 ${pi/2} 0"/>
-      <geometry>
-        <cylinder length="${color_camera_thickness}" radius="${color_camera_diameter/2}"/>
-      </geometry>
-      <material name="white"/>
-    </visual>
-  </link>
-  <joint name="imu_joint" type="fixed">
-    <parent link="tablet_link"/>
-    <child link="imu_link"/>
-    <origin xyz="${imu_joint_dx} ${imu_joint_dy} ${imu_joint_dz+tablet_height/2}" rpy="0 0 0"/>
-  </joint>
-  <link name="imu_link">
-    <visual>
-      <origin xyz="0 0 0" rpy="0 0 0"/>
-      <geometry>
-        <box size="${imu_xlen} ${imu_ylen} ${imu_zlen}"/>
-      </geometry>
-      <material name="black"/>
-    </visual>
-  </link>
-  <gazebo reference="color_camera_link">
-    <sensor type="camera" name="color_camera">
-      <always_on>true</always_on>
-      <visualize>false</visualize>
-      <update_rate>15.0</update_rate>
-      <camera name="front_color_camera">
-        <horizontal_fov>1.3962634</horizontal_fov>
-        <image>
-          <width>720</width>
-          <height>480</height>
-          <format>R8G8B8</format>
-        </image>
-        <clip>
-          <near>0.02</near>
-          <far>300</far>
-        </clip>
-        <noise>
-          <type>gaussian</type>
-          <mean>0.0</mean>
-          <stddev>0.007</stddev>
-        </noise>
-      </camera>
-      <plugin name="color_camera_plugin" filename="libgazebo_ros_camera.so">
-        <!-- ros -->
-          <!-- remapping -->
-          <!-- namespace -->
-        <!-- /ros -->
-        <!-- camera_name>omit, defaults to sensor name</camera_name -->
-        <!-- frame_name>omit, defaults to link name</frameName -->
-        <!-- hack_baseline>0.07</hack_baseline -->
-      </plugin>
-    </sensor>
-  </gazebo>
   <gazebo>
     <plugin name="differential_drive_plugin" filename="libgazebo_ros_diff_drive.so">

Commit message: URDF edit

File: urdf/robot.urdf.xacro (robot description, xacro)
@@ -11,23 +11,21 @@
   <xacro:property name="caster_diameter" value="0.017"/>
   <!-- Caster center to base edge -->
-  <xacro:property name="caster_inset" value="0.0386"/>
+  <xacro:property name="caster_inset" value="0.011"/>
   <xacro:property name="floor_clearance" value="0.0149"/>
   <xacro:property name="base_diameter" value="0.124"/>
   <xacro:property name="wheel_base" value="0.105043"/>
-  <xacro:property name="lower_cylinder_height" value="0.1227"/>
-  <xacro:property name="lower_to_upper_cylinders_gap" value="0.0195"/>
-  <xacro:property name="laser_puck_to_upper_cylinder_gap" value="0.0022"/>
-  <xacro:property name="laser_puck_diameter" value="0.0656"/>
-  <xacro:property name="upper_cylinder_height" value="0.003"/>
+  <xacro:property name="lower_cylinder_height" value="0.032"/>
+  <xacro:property name="laser_puck_height" value="0.016"/>
+  <xacro:property name="laser_puck_diameter" value="0.06"/>
+  <xacro:property name="laser_puck_offset" value="0.0384"/>
   <xacro:property name="head_height" value="0.09"/>
   <!-- N*m -->
   <xacro:property name="motor_stall_torque" value="0.171616375"/>
   <xacro:property name="max_wheel_acceleration" value="1"/>
-  <xacro:property name="lower_cylinder_mass" value="0.500"/>
+  <xacro:property name="lower_cylinder_mass" value="0.250"/>
   <!-- caster and battery weight -->
-  <xacro:property name="caster_mass" value="0.420"/>
+  <xacro:property name="caster_mass" value="0.050"/>
   <xacro:property name="wheel_mass" value="0.050"/>
   <xacro:property name="laser_puck_mass" value="0.200"/>
-  <xacro:property name="upper_cylinder_mass" value="0.100"/>
   <xacro:property name="head_mass" value="0.200"/>
   <!-- ****************** **************** ****************** -->
@@ -215,5 +213,5 @@
     <parent link="base_link"/>
     <child link="base_scan"/>
-    <origin xyz="0 0 ${lower_cylinder_height + (lower_to_upper_cylinders_gap - laser_puck_to_upper_cylinder_gap)/2}" rpy="-${pi} 0 0"/>
+    <origin xyz="0 0 ${lower_cylinder_height + laser_puck_offset}" rpy="-${pi} 0 0"/>
   </joint>
   <link name="base_scan">
@@ -221,5 +219,5 @@
       <origin xyz="0 0 0" rpy="0 0 0"/>
       <geometry>
-        <cylinder length="${lower_to_upper_cylinders_gap - laser_puck_to_upper_cylinder_gap}" radius="${laser_puck_diameter/2}"/>
+        <cylinder length="${laser_puck_height}" radius="${laser_puck_diameter/2}"/>
       </geometry>
       <material name="blue"/>
@@ -228,34 +226,13 @@
       <origin xyz="0 0 0" rpy="0 0 0"/>
       <geometry>
-        <cylinder length="${lower_to_upper_cylinders_gap - laser_puck_to_upper_cylinder_gap}" radius="${laser_puck_diameter/2}"/>
-      </geometry>
-    </collision>
-    <xacro:solid_cylinder_inertia m="${laser_puck_mass}" r="${laser_puck_diameter/2}" h="${lower_to_upper_cylinders_gap - laser_puck_to_upper_cylinder_gap}"/>
-  </link>
-  <joint name="base_upper_joint" type="fixed">
-    <parent link="base_link"/>
-    <child link="base_upper_link"/>
-    <origin xyz="0 0 ${lower_cylinder_height + lower_to_upper_cylinders_gap}" rpy="0 0 0"/>
-  </joint>
-  <link name="base_upper_link">
-    <visual>
-      <origin xyz="0 0 ${upper_cylinder_height/2}" rpy="0 0 0"/>
-      <geometry>
-        <cylinder length="${upper_cylinder_height}" radius="${base_diameter/2}"/>
-      </geometry>
-      <material name="white"/>
-    </visual>
-    <collision>
-      <origin xyz="0 0 ${upper_cylinder_height/2}" rpy="0 0 0"/>
-      <geometry>
-        <cylinder length="${upper_cylinder_height}" radius="${base_diameter/2}"/>
-      </geometry>
-    </collision>
-    <xacro:solid_cylinder_inertia m="${upper_cylinder_mass}" r="${base_diameter/2}" h="${upper_cylinder_height}"/>
+        <cylinder length="${laser_puck_height}" radius="${laser_puck_diameter/2}"/>
+      </geometry>
+    </collision>
+    <xacro:solid_cylinder_inertia m="${laser_puck_mass}" r="${laser_puck_diameter/2}" h="${laser_puck_height}"/>
   </link>
   <joint name="head_joint" type="fixed">
-    <parent link="base_upper_link"/>
+    <parent link="base_link"/>
     <child link="head_link"/>
-    <origin xyz="0 0 ${upper_cylinder_height}" rpy="0 0 0"/>
+    <origin xyz="0 0 ${lower_cylinder_height}" rpy="0 0 0"/>
   </joint>
   <link name="head_link">
@@ -350,61 +327,4 @@
     </sensor>
   </gazebo>
-  <gazebo reference="imu_link">
-    <gravity>true</gravity>
-    <sensor name="imu_sensor" type="imu">
-      <always_on>true</always_on>
-      <update_rate>100</update_rate>
-      <!-- visualize>true</visualize -->
-      <imu>
-        <angular_velocity>
-          <x>
-            <noise type="gaussian">
-              <mean>0.0</mean>
-              <stddev>2e-4</stddev>
-            </noise>
-          </x>
-          <y>
-            <noise type="gaussian">
-              <mean>0.0</mean>
-              <stddev>2e-4</stddev>
-            </noise>
-          </y>
-          <z>
-            <noise type="gaussian">
-              <mean>0.0</mean>
-              <stddev>2e-4</stddev>
-            </noise>
-          </z>
-        </angular_velocity>
-        <linear_acceleration>
-          <x>
-            <noise type="gaussian">
-              <mean>0.0</mean>
-              <stddev>1.7e-2</stddev>
-            </noise>
-          </x>
-          <y>
-            <noise type="gaussian">
-              <mean>0.0</mean>
-              <stddev>1.7e-2</stddev>
-            </noise>
-          </y>
-          <z>
-            <noise type="gaussian">
-              <mean>0.0</mean>
-              <stddev>1.7e-2</stddev>
-            </noise>
-          </z>
-        </linear_acceleration>
-      </imu>
-      <!-- https://github.com/ros-simulation/gazebo_ros_pkgs/blob/foxy/gazebo_plugins/src/gazebo_ros_imu_sensor.cpp -->
-      <plugin filename="libgazebo_ros_imu_sensor.so" name="imu_plugin">
-        <ros>
-          <!-- namespace>/robot_instance_1</namespace -->
-          <remapping>~/out:=imu</remapping>
-        </ros>
-      </plugin>
-    </sensor>
-  </gazebo>
   <gazebo reference="wheel_left_link">
     <mu1>0.2</mu1>

Commit message: URDF edit

File: urdf/robot.urdf.xacro (robot description, xacro)
@@ -19,5 +19,5 @@
   <xacro:property name="laser_puck_diameter" value="0.06"/>
   <xacro:property name="laser_puck_offset" value="0.0384"/>
-  <xacro:property name="head_height" value="0.09"/>
+  <xacro:property name="head_height" value="0.0388"/>
   <!-- N*m -->
   <xacro:property name="motor_stall_torque" value="0.171616375"/>
@@ -240,5 +240,5 @@
       <origin xyz="0 0 0" rpy="0 0 0"/>
       <geometry>
-        <mesh filename="package://makerspet_mini/mesh/head.stl" scale="${0.001*base_diameter} ${0.001*base_diameter} ${0.001*head_height*2}"/>
+        <mesh filename="package://makerspet_mini/mesh/hemisphere.stl" scale="${0.001*base_diameter} ${0.001*base_diameter} ${0.001*head_height*2}"/>
       </geometry>
       <material name="red"/>

Commit message: URDF colors, scan rate

File: urdf/robot.urdf.xacro (robot description, xacro)
@@ -156,5 +156,5 @@
         <sphere radius="${caster_diameter/2}"/>
       </geometry>
-      <material name="yellow"/>
+      <material name="white"/>
     </visual>
    <collision>
@@ -178,5 +178,5 @@
         <cylinder length="${wheel_width}" radius="${wheel_diameter/2}"/>
       </geometry>
-      <material name="blue"/>
+      <material name="red"/>
     </visual>
     <collision>
@@ -200,5 +200,5 @@
         <cylinder length="${wheel_width}" radius="${wheel_diameter/2}"/>
       </geometry>
-      <material name="blue"/>
+      <material name="red"/>
     </visual>
     <collision>
@@ -212,5 +212,5 @@
   <joint name="scan_joint" type="fixed">
     <parent link="base_link"/>
-    <child link="base_scan"/>
+    <child link="base_scan_link"/>
     <origin xyz="0 0 ${lower_cylinder_height + laser_puck_offset}" rpy="-${pi} 0 0"/>
   </joint>
@@ -221,5 +221,5 @@
         <cylinder length="${laser_puck_height}" radius="${laser_puck_diameter/2}"/>
       </geometry>
-      <material name="blue"/>
+      <material name="black"/>
     </visual>
     <collision>
@@ -293,5 +293,5 @@
       <visualize>false</visualize>
       <always_on>true</always_on>
-      <update_rate>9</update_rate>
+      <update_rate>5</update_rate>
       <ray>
         <scan>
@@ -305,5 +305,5 @@
         <range>
           <min>0.1</min>
-          <max>12.0</max>
+          <max>10.0</max>
           <resolution>0.02</resolution>
         </range>
@@ -332,5 +332,5 @@
     <!-- mu>100000.0</mu -->
     <!-- mu2>100000.0</mu2 -->
-    <material>Gazebo/Blue</material>
+    <material>Gazebo/Red</material>
     <!-- fdir1>0 0 0</fdir1 -->
     <!-- kp>1e+5</kp -->
@@ -347,10 +347,10 @@
     <mu1>0.2</mu1>
     <mu2>0.2</mu2>
-    <material>Gazebo/Blue</material>
+    <material>Gazebo/Red</material>
   </gazebo>
   <gazebo reference="caster_link">
     <mu1>0.2</mu1>
     <mu2>0.2</mu2>
-    <material>Gazebo/Yellow</material>
+    <material>Gazebo/White</material>
   </gazebo>
   <gazebo reference="head_link">
@@ -360,6 +360,6 @@
     <material>Gazebo/White</material>
   </gazebo>
-  <gazebo reference="base_upper_link">
-    <material>Gazebo/White</material>
+  <gazebo reference="base_scan">
+    <material>Gazebo/Black</material>
   </gazebo>
 </robot>

Commit message: SDF

File: urdf/robot.urdf.xacro (robot description, xacro)
@@ -212,5 +212,5 @@
   <joint name="scan_joint" type="fixed">
     <parent link="base_link"/>
-    <child link="base_scan_link"/>
+    <child link="base_scan"/>
     <origin xyz="0 0 ${lower_cylinder_height + laser_puck_offset}" rpy="-${pi} 0 0"/>
   </joint>

Commit message: LiDAR orientation

File: urdf/robot.urdf.xacro (robot description, xacro)
@@ -213,5 +213,5 @@
     <parent link="base_link"/>
     <child link="base_scan"/>
-    <origin xyz="0 0 ${lower_cylinder_height + laser_puck_offset}" rpy="-${pi} 0 0"/>
+    <origin xyz="0 0 ${lower_cylinder_height + laser_puck_offset}" rpy="0 0 -${pi}"/>
   </joint>
   <link name="base_scan">

Commit message: LiDAR orientation fix

File: urdf/robot.urdf.xacro (robot description, xacro)
@@ -213,5 +213,5 @@
     <parent link="base_link"/>
     <child link="base_scan"/>
-    <origin xyz="0 0 ${lower_cylinder_height + laser_puck_offset}" rpy="0 0 -${pi}"/>
+    <origin xyz="0 0 ${lower_cylinder_height + laser_puck_offset}" rpy="0 -${pi} 0"/>
   </joint>
   <link name="base_scan">

Commit message: URDF caster fix

File: urdf/robot.urdf.xacro (robot description, xacro)
@@ -20,4 +20,5 @@
   <xacro:property name="laser_puck_offset" value="0.0384"/>
   <xacro:property name="head_height" value="0.0388"/>
+  <xacro:property name="lidar_center_offset" value="0"/>
   <!-- N*m -->
   <xacro:property name="motor_stall_torque" value="0.171616375"/>
@@ -148,5 +149,5 @@
     <parent link="base_link"/>
     <child link="caster_link"/>
-    <origin xyz="${base_diameter/2-caster_inset} 0 ${caster_diameter/2-floor_clearance}" rpy="0 0 0"/>
+    <origin xyz="${caster_inset-base_diameter/2} 0 ${caster_diameter/2-floor_clearance}" rpy="0 0 0"/>
   </joint>
   <link name="caster_link">
@@ -213,5 +214,5 @@
     <parent link="base_link"/>
     <child link="base_scan"/>
-    <origin xyz="0 0 ${lower_cylinder_height + laser_puck_offset}" rpy="0 -${pi} 0"/>
+    <origin xyz="${lidar_center_offset} 0 ${lower_cylinder_height + laser_puck_offset}" rpy="0 -${pi} 0"/>
   </joint>
   <link name="base_scan">

Commit message: Reduced min angular speed

File: urdf/robot.urdf.xacro (robot description, xacro)
@@ -20,5 +20,5 @@
   <xacro:property name="laser_puck_offset" value="0.0384"/>
   <xacro:property name="head_height" value="0.0388"/>
-  <xacro:property name="lidar_center_offset" value="0"/>
+  <xacro:property name="lidar_center_offset" value="0.000"/>
   <!-- N*m -->
   <xacro:property name="motor_stall_torque" value="0.171616375"/>

Commit message: URDF LiDAR motor

File: urdf/robot.urdf.xacro (robot description, xacro)
@@ -19,4 +19,8 @@
   <xacro:property name="laser_puck_diameter" value="0.06"/>
   <xacro:property name="laser_puck_offset" value="0.0384"/>
+  <xacro:property name="laser_motor_diameter" value="0.02"/>
+  <xacro:property name="lidar_motor_x_offset" value="0.04"/>
+  <xacro:property name="lidar_motor_z_offset" value="0.012"/>
+  <xacro:property name="laser_motor_height" value="0.01"/>
   <xacro:property name="head_height" value="0.0388"/>
   <xacro:property name="lidar_center_offset" value="0.000"/>
@@ -28,5 +32,6 @@
   <xacro:property name="caster_mass" value="0.050"/>
   <xacro:property name="wheel_mass" value="0.050"/>
-  <xacro:property name="laser_puck_mass" value="0.200"/>
+  <xacro:property name="laser_puck_mass" value="0.150"/>
+  <xacro:property name="laser_motor_mass" value="0.050"/>
   <xacro:property name="head_mass" value="0.200"/>
   <!-- ****************** **************** ****************** -->
@@ -231,4 +236,25 @@
     </collision>
     <xacro:solid_cylinder_inertia m="${laser_puck_mass}" r="${laser_puck_diameter/2}" h="${laser_puck_height}"/>
+  </link>
+  <joint name="scan_motor_joint" type="fixed">
+    <parent link="base_scan"/>
+    <child link="scan_motor"/>
+    <origin xyz="${lidar_motor_x_offset} 0 ${lidar_motor_z_offset}" rpy="0 -${pi} 0"/>
+  </joint>
+  <link name="scan_motor">
+    <visual>
+      <origin xyz="0 0 0" rpy="0 0 0"/>
+      <geometry>
+        <cylinder length="${laser_motor_height}" radius="${laser_motor_diameter/2}"/>
+      </geometry>
+      <material name="black"/>
+    </visual>
+    <collision>
+      <origin xyz="0 0 0" rpy="0 0 0"/>
+      <geometry>
+        <cylinder length="${laser_motor_height}" radius="${laser_motor_diameter/2}"/>
+      </geometry>
+    </collision>
+    <xacro:solid_cylinder_inertia m="${laser_motor_mass}" r="${laser_motor_diameter/2}" h="${laser_motor_height}"/>
   </link>
   <joint name="head_joint" type="fixed">
