Commit message: Gazebo Ignition before debug

File: urdf/robot.urdf.xacro (robot description, xacro)
@@ -1,131 +1,8 @@
 <?xml version="1.0" ?>
 <robot name="makerspet_mini" xmlns:xacro="http://ros.org/wiki/xacro">
-  <!-- https://classic.gazebosim.org/tutorials?tut=ros_gzplugins&cat=connect_ros -->
-  <!-- https://classic.gazebosim.org/tutorials?tut=ros_urdf&cat=connect_ros -->
-  <!-- https://github.com/ROBOTIS-GIT/turtlebot3_simulations/blob/humble-devel/turtlebot3_gazebo/models/turtlebot3_waffle_pi/model.sdf -->
-  <!-- https://github.com/ROBOTIS-GIT/turtlebot3/blob/humble-devel/turtlebot3_description/urdf/turtlebot3_waffle_pi.urdf -->
-  <!-- ****************** ROBOT DIMENSIONS ****************** -->
-  <!-- Units: meters, degrees, kg, N*m, m/s2 -->
-  <xacro:property name="wheel_diameter" value="0.043"/>
-  <xacro:property name="wheel_width" value="0.0055"/>
-  <xacro:property name="caster_diameter" value="0.017"/>
-  <!-- Caster center to base edge -->
-  <xacro:property name="caster_inset" value="0.011"/>
-  <xacro:property name="floor_clearance" value="0.0149"/>
-  <xacro:property name="base_diameter" value="0.124"/>
-  <xacro:property name="wheel_base" value="0.105043"/>
-  <xacro:property name="lower_cylinder_height" value="0.032"/>
-  <xacro:property name="laser_puck_height" value="0.016"/>
-  <xacro:property name="laser_puck_diameter" value="0.06"/>
-  <xacro:property name="laser_puck_offset" value="0.0384"/>
-  <xacro:property name="laser_motor_diameter" value="0.02"/>
-  <xacro:property name="lidar_motor_x_offset" value="0.04"/>
-  <xacro:property name="lidar_motor_z_offset" value="0.012"/>
-  <xacro:property name="laser_motor_height" value="0.01"/>
-  <xacro:property name="head_height" value="0.0388"/>
-  <xacro:property name="lidar_center_offset" value="0.000"/>
-  <!-- N*m -->
-  <xacro:property name="motor_stall_torque" value="0.171616375"/>
-  <xacro:property name="max_wheel_acceleration" value="1"/>
-  <xacro:property name="lower_cylinder_mass" value="0.250"/>
-  <!-- caster and battery weight -->
-  <xacro:property name="caster_mass" value="0.050"/>
-  <xacro:property name="wheel_mass" value="0.050"/>
-  <xacro:property name="laser_puck_mass" value="0.150"/>
-  <xacro:property name="laser_motor_mass" value="0.050"/>
-  <xacro:property name="head_mass" value="0.200"/>
-  <!-- ****************** **************** ****************** -->
-  <xacro:property name="DEG2RAD" value="0.0174533"/>
-  <material name="black">
-      <color rgba="0 0 0 1.0"/>
-  </material>
-  <material name="dark">
-    <color rgba="0.3 0.3 0.3 1.0"/>
-  </material>
-  <material name="light_black">
-    <color rgba="0.4 0.4 0.4 1.0"/>
-  </material>
-  <material name="blue">
-    <color rgba="0 0 0.8 1.0"/>
-  </material>
-  <material name="green">
-    <color rgba="0 0.8 0 1.0"/>
-  </material>
-  <material name="grey">
-    <color rgba="0.5 0.5 0.5 1.0"/>
-  </material>
-  <material name="orange">
-    <color rgba="1.0 0.4235 0.0392 1.0"/>
-  </material>
-  <material name="brown">
-    <color rgba="0.8706 0.8118 0.7647 1.0"/>
-  </material>
-  <material name="red">
-    <color rgba="0.8 0 0 1.0"/>
-  </material>
-  <material name="yellow">
-    <color rgba="0.8 0.8 0 1.0"/>
-  </material>
-  <material name="white">
-    <color rgba="1.0 1.0 1.0 1.0"/>
-  </material>
-  <xacro:macro name="solid_box_inertia" params="m x y z">
-    <inertial>
-      <origin xyz="0 0 0" rpy="${pi/2} 0 ${pi/2}"/>
-      <mass value="${m}"/>
-      <inertia ixx="${m*(y*y+z*z)/12}" ixy="0" ixz="0" iyy="${m*(x*x+z*z)/12}" iyz="0" izz="${m*(x*x+y*y)/12}"/>
-    </inertial>
-  </xacro:macro>
-  <xacro:macro name="solid_cylinder_inertia" params="m r h">
-    <inertial>
-      <origin xyz="0 0 0" rpy="${pi/2} 0 0" />
-      <mass value="${m}"/>
-      <inertia ixx="${m*(3*r*r+h*h)/12}" ixy="0" ixz="0" iyy="${m*(3*r*r+h*h)/12}" iyz="0" izz="${m*r*r/2}"/>
-    </inertial>
-  </xacro:macro>
-  <xacro:macro name="hollow_cylinder_inertia" params="m ri ro h">
-    <inertial>
-      <origin xyz="0 0 0" rpy="${pi/2} 0 0" />
-      <mass value="${m}"/>
-      <inertia ixx="${m*(3*(ri*ri+ro*ro)+h*h)/12}" ixy="0" ixz="0" iyy="${m*(3*(ri*ri+ro*ro) + h*h)/12}" iyz="0" izz="${m*(ri*ri+ro*ro)/2}"/>
-    </inertial>
-  </xacro:macro>
-  <xacro:macro name="thin_cylindrical_shell_inertia" params="m r h">
-    <inertial>
-      <origin xyz="0 0 0" rpy="${pi/2} 0 0" />
-      <mass value="${m}"/>
-      <inertia ixx="${m*(6*r*r+h*h)/12}" ixy="0" ixz="0" iyy="${m*(6*r*r+h*h)/12}" iyz="0" izz="${m*r*r}"/>
-    </inertial>
-  </xacro:macro>
-  <xacro:macro name="solid_sphere_inertia" params="m r">
-    <inertial>
-      <mass value="${m}"/>
-      <inertia ixx="${2*m*r*r/5}" ixy="0" ixz="0" iyy="${2*m*r*r/5}" iyz="0" izz="${2*m*r*r/5}"/>
-    </inertial>
-  </xacro:macro>
-  <xacro:macro name="thin_spherical_shell_inertia" params="m r">
-    <inertial>
-      <mass value="${m}"/>
-      <inertia ixx="${2*m*r*r/3}" ixy="0" ixz="0" iyy="${2*m*r*r/3}" iyz="0" izz="${2*m*r*r/3}"/>
-    </inertial>
-  </xacro:macro>
-  <xacro:macro name="solid_hemisphere_inertia" params="m r">
-    <inertial>
-      <mass value="${m}"/>
-      <inertia ixx="${83*m*r*r/320}" ixy="0" ixz="0" iyy="${83*m*r*r/320}" iyz="0" izz="${2*m*r*r/5}"/>
-    </inertial>
-  </xacro:macro>
-  <xacro:macro name="solid_ellipsoid_inertia" params="m x y z">
-    <inertial>
-      <mass value="${m}"/>
-      <inertia ixx="${m*(y*y+z*z)/5}" ixy="0" ixz="0" iyy="${m*(x*x+z*z)/5}" iyz="0" izz="${m*(x*x+y*y)/5}"/>
-    </inertial>
-  </xacro:macro>
-  <xacro:macro name="solid_semi_ellipsoid_inertia" params="m x y z">
-    <inertial>
-      <mass value="${m}"/>
-      <inertia ixx="${m*(y*y+z*z)/10}" ixy="0" ixz="0" iyy="${m*(x*x+z*z)/10}" iyz="0" izz="${m*(x*x+y*y)/10}"/>
-    </inertial>
-  </xacro:macro>
+  <xacro:include filename="params.xacro" />
+  <xacro:include filename="inertial.xacro" />
+  <xacro:include filename="plugins.xacro" />
+  <xacro:include filename="materials.xacro" />
   <!-- ****************** **************** ****************** -->
   <link name="base_footprint"/>
@@ -279,114 +156,3 @@
     <xacro:solid_semi_ellipsoid_inertia m="${head_mass}" x="${base_diameter/2}" y="${base_diameter/2}" z="${head_height}"/>
   </link>
-  <gazebo>
-    <plugin name="differential_drive_plugin" filename="libgazebo_ros_diff_drive.so">
-      <!-- /opt/ros/humble/share/gazebo_plugins/worlds/gazebo_ros_diff_drive_demo.world -->
-      <!-- https://github.com/ros-simulation/gazebo_ros_pkgs/blob/foxy/gazebo_plugins/src/gazebo_ros_diff_drive.cpp -->
-      <!-- ros -->
-        <!-- remapping -->
-        <!-- namespace -->
-      <!-- /ros -->
-      <update_rate>30</update_rate>
-      <left_joint>wheel_left_joint</left_joint>
-      <right_joint>wheel_right_joint</right_joint>
-      <wheel_separation>${wheel_base}</wheel_separation>
-      <wheel_diameter>${wheel_diameter}</wheel_diameter>
-      <max_wheel_torque>${motor_stall_torque}</max_wheel_torque>
-      <max_wheel_acceleration>${max_wheel_acceleration}</max_wheel_acceleration>
-      <command_topic>cmd_vel</command_topic>
-      <publish_odom>true</publish_odom>
-      <publish_odom_tf>true</publish_odom_tf>
-      <publish_wheel_tf>false</publish_wheel_tf>
-      <odometry_topic>odom</odometry_topic>
-      <odometry_frame>odom</odometry_frame>
-      <robot_base_frame>base_footprint</robot_base_frame>
-    </plugin>
-  </gazebo>
-  <gazebo>
-    <plugin name="joint_state_plugin" filename="libgazebo_ros_joint_state_publisher.so">
-      <!-- https://github.com/ros-simulation/gazebo_ros_pkgs/blob/foxy/gazebo_plugins/src/gazebo_ros_joint_state_publisher.cpp -->
-      <ros>
-        <!-- namespace -->
-        <remapping>~/out:=joint_states</remapping>
-      </ros>
-      <update_rate>30</update_rate>
-      <joint_name>wheel_left_joint</joint_name>
-      <joint_name>wheel_right_joint</joint_name>
-    </plugin>
-  </gazebo>
-  <gazebo reference="base_scan">
-    <sensor type="ray" name="laser_scan_sensor">
-      <!-- pose>0 0 0 0 0 0</pose -->
-      <visualize>false</visualize>
-      <always_on>true</always_on>
-      <update_rate>5</update_rate>
-      <ray>
-        <scan>
-          <horizontal>
-            <samples>360</samples>
-            <resolution>1</resolution>
-            <min_angle>0</min_angle>
-            <max_angle>${2*pi}</max_angle>
-          </horizontal>
-        </scan>
-        <range>
-          <min>0.1</min>
-          <max>10.0</max>
-          <resolution>0.02</resolution>
-        </range>
-        <noise>
-          <type>gaussian</type>
-          <mean>0.0</mean>
-          <stddev>0.01</stddev>
-        </noise>
-      </ray>
-      <plugin name="laser_scan_plugin" filename="libgazebo_ros_ray_sensor.so">
-        <!-- https://github.com/ros-simulation/gazebo_ros_pkgs/blob/foxy/gazebo_plugins/src/gazebo_ros_ray_sensor.cpp -->
-        <ros>
-          <!-- namespace -->
-          <remapping>~/out:=scan</remapping>
-        </ros>
-        <output_type>sensor_msgs/LaserScan</output_type>
-        <frame_name>base_scan</frame_name>
-        <!-- frameName>base_scan</frameName -->
-        <!-- topicName>/scan</topicName -->
-      </plugin>
-    </sensor>
-  </gazebo>
-  <gazebo reference="wheel_left_link">
-    <mu1>0.2</mu1>
-    <mu2>0.2</mu2>
-    <!-- mu>100000.0</mu -->
-    <!-- mu2>100000.0</mu2 -->
-    <material>Gazebo/Red</material>
-    <!-- fdir1>0 0 0</fdir1 -->
-    <!-- kp>1e+5</kp -->
-    <!-- kd>1</kd -->
-    <!-- min_depth>0.001</min_depth -->
-    <!-- max_vel>0.01</max_vel -->
-    <!-- Turtlebot3 SDF -->
-    <!-- slip1>0.0</slip1 -->
-    <!-- slip2>0.0</slip2 -->
-    <!-- soft_cfm>0</soft_cfm -->
-    <!-- soft_erp>0.2</soft_erp -->
-  </gazebo>
-  <gazebo reference="wheel_right_link">
-    <mu1>0.2</mu1>
-    <mu2>0.2</mu2>
-    <material>Gazebo/Red</material>
-  </gazebo>
-  <gazebo reference="caster_link">
-    <mu1>0.2</mu1>
-    <mu2>0.2</mu2>
-    <material>Gazebo/White</material>
-  </gazebo>
-  <gazebo reference="head_link">
-    <material>Gazebo/Red</material>
-  </gazebo>
-  <gazebo reference="base_link">
-    <material>Gazebo/White</material>
-  </gazebo>
-  <gazebo reference="base_scan">
-    <material>Gazebo/Black</material>
-  </gazebo>
 </robot>
