Commit message: Gazebo Ignition debug

File: urdf/inertial.xacro (robot description, xacro)
@@ -20,5 +20,6 @@
       <origin xyz="0 0 0" rpy="${pi/2} 0 0" />
       <mass value="${m}"/>
-      <inertia ixx="${m*(3*(ri*ri+ro*ro)+h*h)/12}" ixy="0" ixz="0" iyy="${m*(3*(ri*ri+ro*ro) + h*h)/12}" iyz="0" izz="$>    </inertial>
+      <inertia ixx="${m*(3*(ri*ri+ro*ro)+h*h)/12}" ixy="0" ixz="0" iyy="${m*(3*(ri*ri+ro*ro) + h*h)/12}" iyz="0" izz="${m*(ri*ri+ro*ro)/2}"/>
+    </inertial>
   </xacro:macro>
   <xacro:macro name="thin_cylindrical_shell_inertia" params="m r h">

File: urdf/materials.xacro (robot description, xacro)
@@ -1,4 +1,4 @@
 <?xml version="1.0"?>
-<robot>
+<robot xmlns:xacro="http://ros.org/wiki/xacro">
   <material name="black">
       <color rgba="0 0 0 1.0"/>

File: urdf/params.xacro (robot description, xacro)
@@ -1,4 +1,4 @@
 <?xml version="1.0" ?>
-<robot>
+<robot xmlns:xacro="http://ros.org/wiki/xacro">
   <!-- ****************** ROBOT DIMENSIONS ****************** -->
   <!-- Units: meters, degrees, kg, N*m, m/s2 -->

File: urdf/plugins.xacro (robot description, xacro)
@@ -1,4 +1,4 @@
 <?xml version="1.0"?>
-<robot>
+<robot xmlns:xacro="http://ros.org/wiki/xacro">
   <gazebo>
     <plugin filename="gz-sim-diff-drive-system" name="gz::sim::systems::DiffDrive">
@@ -41,4 +41,5 @@
   <gazebo reference="base_scan">
     <!-- sensor name="laser" type="gpu_lidar" -->
+    <sensor type="ray" name="laser_scan_sensor">
     <!-- pose> 0 0 0 0 0 0 </pose -->
     <visualize>false</visualize>
