Commit message: Migrate max wheel torque

File: urdf/params.xacro (robot description, xacro)
@@ -23,5 +23,5 @@
   <!-- N*m -->
   <xacro:property name="motor_stall_torque" value="0.171616375"/>
-  <xacro:property name="max_wheel_acceleration" value="1"/>
+  <xacro:property name="max_linear_acceleration" value="1"/>
   <xacro:property name="lower_cylinder_mass" value="0.250"/>
   <!-- caster and battery weight -->

File: urdf/plugins.xacro (robot description, xacro)
@@ -1,3 +1,6 @@
 <?xml version="1.0"?>
+<!-- https://gazebosim.org/docs/latest/migrating_gazebo_classic_ros2_packages/ -->
+<!-- Turtlebot3 Jazzy https://emanual.robotis.com/docs/en/platform/turtlebot3/simulation/ -->
+<!-- Build URDF xacro robot.urdf.xacro -->
 <robot xmlns:xacro="http://ros.org/wiki/xacro">
   <gazebo>
@@ -7,6 +10,5 @@
       <wheel_separation>${wheel_base}</wheel_separation>
       <wheel_radius>${wheel_diameter/2}</wheel_radius>
-      <max_wheel_torque>${motor_stall_torque}</max_wheel_torque>
-      <max_wheel_acceleration>${max_wheel_acceleration}</max_wheel_acceleration>
+      <max_linear_acceleration>${max_linear_acceleration}</max_linear_acceleration>
       <!-- update_rate>30</update_rate -->
       <!-- command_topic>cmd_vel</command_topic -->
@@ -17,7 +19,4 @@
       <!-- odometry_frame>odom</odometry_frame -->
       <!-- robot_base_frame>base_footprint</robot_base_frame -->
-      <!-- wheel_separation>0.35</wheel_separation -->
-      <!-- wheel_radius>0.05</wheel_radius -->
-      <!-- max_linear_acceleration>10</max_linear_acceleration -->
       <topic>cmd_vel</topic>
     </plugin>
@@ -30,4 +29,7 @@
       <tf_topic>/tf</tf_topic>
       <dimensions>2</dimensions>
+      <!-- topic>joint_states</topic --> <!--from <ros><remapping> -->
+      <!-- joint_name>wheel_left_joint</joint_name -->
+      <!-- joint_name>wheel_right_joint</joint_name -->
     </plugin>
     <plugin filename="gz-sim-joint-state-publisher-system" name="gz::sim::systems::JointStatePublisher">

File: urdf/robot.urdf.xacro (robot description, xacro)
@@ -51,5 +51,9 @@
     <child link="wheel_left_link"/>
     <origin xyz="0 ${wheel_base/2} ${wheel_diameter/2-floor_clearance}" rpy="-${pi/2} 0 0"/>
-    <axis xyz="0 0 1"/>
+    <axis xyz="0 0 1">
+      <limit>
+        <effort>${motor_stall_torque}</effort>
+      </limit>
+    </axis>
   </joint>
   <link name="wheel_left_link">
@@ -72,5 +76,9 @@
     <child link="wheel_right_link"/>
     <origin xyz="0 ${-wheel_base/2} ${wheel_diameter/2-floor_clearance}" rpy="-${pi/2} 0 0"/>
-    <axis xyz="0 0 1"/>
+    <axis xyz="0 0 1">
+      <limit>
+        <effort>${motor_stall_torque}</effort>
+      </limit>
+    </axis>
   </joint>
   <link name="wheel_right_link">
