Commit message: Fix color warnings

File: urdf/materials.xacro (robot description, xacro)
@@ -1,37 +1,4 @@
 <?xml version="1.0"?>
 <robot xmlns:xacro="http://ros.org/wiki/xacro">
-  <material name="black">
-      <color rgba="0 0 0 1.0"/>
-  </material>
-  <material name="dark">
-    <color rgba="0.3 0.3 0.3 1.0"/>
-  </material>
-  <material name="light_black">
-    <color rgba="0.4 0.4 0.4 1.0"/>
-  </material>
-  <material name="blue">
-    <color rgba="0 0 0.8 1.0"/>
-  </material>
-  <material name="green">
-    <color rgba="0 0.8 0 1.0"/>
-  </material>
-  <material name="grey">
-    <color rgba="0.5 0.5 0.5 1.0"/>
-  </material>
-  <material name="orange">
-    <color rgba="1.0 0.4235 0.0392 1.0"/>
-  </material>
-  <material name="brown">
-    <color rgba="0.8706 0.8118 0.7647 1.0"/>
-  </material>
-  <material name="red">
-    <color rgba="0.8 0 0 1.0"/>
-  </material>
-  <material name="yellow">
-    <color rgba="0.8 0.8 0 1.0"/>
-  </material>
-  <material name="white">
-    <color rgba="1.0 1.0 1.0 1.0"/>
-  </material>
   <gazebo reference="wheel_left_link">
     <mu1>0.2</mu1>
@@ -39,5 +6,11 @@
     <!-- mu>100000.0</mu -->
     <!-- mu2>100000.0</mu2 -->
-    <material>Gazebo/Red</material>
+    <visual>
+      <material>
+        <ambient>0.8 0 0 1</ambient>
+        <diffuse>0.8 0 0 1</diffuse>
+        <specular>0.8 0 0 1</specular>
+      </material>
+    </visual>
     <!-- fdir1>0 0 0</fdir1 -->
     <!-- kp>1e+5</kp -->
@@ -54,19 +27,49 @@
     <mu1>0.2</mu1>
     <mu2>0.2</mu2>
-    <material>Gazebo/Red</material>
+    <visual>
+      <material>
+        <ambient>0.8 0 0 1</ambient>
+        <diffuse>0.8 0 0 1</diffuse>
+        <specular>0.8 0 0 1</specular>
+      </material>
+    </visual>
   </gazebo>
   <gazebo reference="caster_link">
     <mu1>0.2</mu1>
     <mu2>0.2</mu2>
-    <material>Gazebo/White</material>
+    <visual>
+      <material>
+        <ambient>1 1 1 1</ambient>
+        <diffuse>1 1 1 1</diffuse>
+        <specular>1 1 1 1</specular>
+      </material>
+    </visual>
   </gazebo>
   <gazebo reference="head_link">
-    <material>Gazebo/Red</material>
+    <visual>
+      <material>
+        <ambient>0.8 0 0 1</ambient>
+        <diffuse>0.8 0 0 1</diffuse>
+        <specular>0.8 0 0 1</specular>
+      </material>
+    </visual>
   </gazebo>
   <gazebo reference="base_link">
-    <material>Gazebo/White</material>
+    <visual>
+      <material>
+        <ambient>1 1 1 1</ambient>
+        <diffuse>1 1 1 1</diffuse>
+        <specular>1 1 1 1</specular>
+      </material>
+    </visual>
   </gazebo>
   <gazebo reference="base_scan">
-    <material>Gazebo/Black</material>
+    <visual>
+      <material>
+        <ambient>0 0 0 1</ambient>
+        <diffuse>0 0 0 1</diffuse>
+        <specular>0 0 0 1</specular>
+      </material>
+    </visual>
   </gazebo>
 </robot>

File: urdf/robot.urdf.xacro (robot description, xacro)
@@ -18,5 +18,4 @@
         <cylinder length="${lower_cylinder_height}" radius="${base_diameter/2}"/>
       </geometry>
-      <material name="white"/>
     </visual>
     <collision>
@@ -39,5 +38,4 @@
         <sphere radius="${caster_diameter/2}"/>
       </geometry>
-      <material name="white"/>
     </visual>
    <collision>
@@ -61,5 +59,4 @@
         <cylinder length="${wheel_width}" radius="${wheel_diameter/2}"/>
       </geometry>
-      <material name="red"/>
     </visual>
     <collision>
@@ -83,5 +80,4 @@
         <cylinder length="${wheel_width}" radius="${wheel_diameter/2}"/>
       </geometry>
-      <material name="red"/>
     </visual>
     <collision>
@@ -104,5 +100,4 @@
         <cylinder length="${laser_puck_height}" radius="${laser_puck_diameter/2}"/>
       </geometry>
-      <material name="black"/>
     </visual>
     <collision>
@@ -125,5 +120,4 @@
         <cylinder length="${laser_motor_height}" radius="${laser_motor_diameter/2}"/>
       </geometry>
-      <material name="black"/>
     </visual>
     <collision>
@@ -146,5 +140,4 @@
         <mesh filename="package://makerspet_mini/mesh/hemisphere.stl" scale="${0.001*base_diameter} ${0.001*base_diameter} ${0.001*head_height*2}"/>
       </geometry>
-      <material name="red"/>
     </visual>
     <collision>

Commit message: Restore non-Gazebo colors

File: urdf/materials.xacro (robot description, xacro)
@@ -1,9 +1,37 @@
 <?xml version="1.0"?>
 <robot xmlns:xacro="http://ros.org/wiki/xacro">
+  <material name="black">
+      <color rgba="0.0 0.0 0.0 1.0"/>
+  </material>
+  <material name="dark">
+    <color rgba="0.3 0.3 0.3 1.0"/>
+  </material>
+  <material name="light_black">
+    <color rgba="0.4 0.4 0.4 1.0"/>
+  </material>
+  <material name="blue">
+    <color rgba="0.0 0.0 0.8 1.0"/>
+  </material>
+  <material name="green">
+    <color rgba="0.0 0.8 0.0 1.0"/>
+  </material>
+  <material name="grey">
+    <color rgba="0.5 0.5 0.5 1.0"/>
+  </material>
+  <material name="orange">
+    <color rgba="1.0 0.4235 0.0392 1.0"/>
+  </material>
+  <material name="brown">
+    <color rgba="0.8706 0.8118 0.7647 1.0"/>
+  </material>
+  <material name="red">
+    <color rgba="0.8 0.0 0.0 1.0"/>
+  </material>
+  <material name="white">
+    <color rgba="1.0 1.0 1.0 1.0"/>
+  </material>
   <gazebo reference="wheel_left_link">
     <mu1>0.2</mu1>
     <mu2>0.2</mu2>
-    <!-- mu>100000.0</mu -->
-    <!-- mu2>100000.0</mu2 -->
     <visual>
       <material>
@@ -13,14 +41,4 @@
       </material>
     </visual>
-    <!-- fdir1>0 0 0</fdir1 -->
-    <!-- kp>1e+5</kp -->
-    <!-- kd>1</kd -->
-    <!-- min_depth>0.001</min_depth -->
-    <!-- max_vel>0.01</max_vel -->
-    <!-- Turtlebot3 SDF -->
-    <!-- slip1>0.0</slip1 -->
-    <!-- slip2>0.0</slip2 -->
-    <!-- soft_cfm>0</soft_cfm -->
-    <!-- soft_erp>0.2</soft_erp -->
   </gazebo>
   <gazebo reference="wheel_right_link">

File: urdf/plugins.xacro (robot description, xacro)
@@ -11,17 +11,8 @@
       <wheel_radius>${wheel_diameter/2}</wheel_radius>
       <max_linear_acceleration>${max_linear_acceleration}</max_linear_acceleration>
-      <!-- update_rate>30</update_rate -->
-      <!-- command_topic>cmd_vel</command_topic -->
-      <!-- publish_odom>true</publish_odom -->
-      <!-- publish_odom_tf>true</publish_odom_tf -->
-      <!-- publish_wheel_tf>false</publish_wheel_tf -->
-      <!-- odometry_topic>odom</odometry_topic -->
-      <!-- odometry_frame>odom</odometry_frame -->
-      <!-- robot_base_frame>base_footprint</robot_base_frame -->
       <topic>cmd_vel</topic>
     </plugin>
     <plugin filename="gz-sim-odometry-publisher-system" name="gz::sim::systems::OdometryPublisher">
       <odom_frame>odom</odom_frame>
-      <!-- robot_base_frame>base_link</robot_base_frame -->
       <robot_base_frame>base_footprint</robot_base_frame>
       <odom_publish_frequency>50</odom_publish_frequency>
@@ -29,7 +20,4 @@
       <tf_topic>/tf</tf_topic>
       <dimensions>2</dimensions>
-      <!-- topic>joint_states</topic --> <!--from <ros><remapping> -->
-      <!-- joint_name>wheel_left_joint</joint_name -->
-      <!-- joint_name>wheel_right_joint</joint_name -->
     </plugin>
     <plugin filename="gz-sim-joint-state-publisher-system" name="gz::sim::systems::JointStatePublisher">

File: urdf/robot.urdf.xacro (robot description, xacro)
@@ -18,4 +18,5 @@
         <cylinder length="${lower_cylinder_height}" radius="${base_diameter/2}"/>
       </geometry>
+      <material name="white"/>
     </visual>
     <collision>
@@ -38,4 +39,5 @@
         <sphere radius="${caster_diameter/2}"/>
       </geometry>
+      <material name="white"/>
     </visual>
    <collision>
@@ -63,4 +65,5 @@
         <cylinder length="${wheel_width}" radius="${wheel_diameter/2}"/>
       </geometry>
+      <material name="red"/>
     </visual>
     <collision>
@@ -88,4 +91,5 @@
         <cylinder length="${wheel_width}" radius="${wheel_diameter/2}"/>
       </geometry>
+      <material name="red"/>
     </visual>
     <collision>
@@ -108,4 +112,5 @@
         <cylinder length="${laser_puck_height}" radius="${laser_puck_diameter/2}"/>
       </geometry>
+      <material name="black"/>
     </visual>
     <collision>
@@ -128,4 +133,5 @@
         <cylinder length="${laser_motor_height}" radius="${laser_motor_diameter/2}"/>
       </geometry>
+      <material name="black"/>
     </visual>
     <collision>
@@ -148,4 +154,5 @@
         <mesh filename="package://makerspet_mini/mesh/hemisphere.stl" scale="${0.001*base_diameter} ${0.001*base_diameter} ${0.001*head_height*2}"/>
       </geometry>
+      <material name="red"/>
     </visual>
     <collision>

Commit message: gz camera works

File: urdf/materials.xacro (robot description, xacro)
@@ -34,60 +34,12 @@
     <mu1>0.2</mu1>
     <mu2>0.2</mu2>
-    <visual>
-      <material>
-        <ambient>0.8 0 0 1</ambient>
-        <diffuse>0.8 0 0 1</diffuse>
-        <specular>0.8 0 0 1</specular>
-      </material>
-    </visual>
   </gazebo>
   <gazebo reference="wheel_right_link">
     <mu1>0.2</mu1>
     <mu2>0.2</mu2>
-    <visual>
-      <material>
-        <ambient>0.8 0 0 1</ambient>
-        <diffuse>0.8 0 0 1</diffuse>
-        <specular>0.8 0 0 1</specular>
-      </material>
-    </visual>
   </gazebo>
   <gazebo reference="caster_link">
     <mu1>0.2</mu1>
     <mu2>0.2</mu2>
-    <visual>
-      <material>
-        <ambient>1 1 1 1</ambient>
-        <diffuse>1 1 1 1</diffuse>
-        <specular>1 1 1 1</specular>
-      </material>
-    </visual>
-  </gazebo>
-  <gazebo reference="head_link">
-    <visual>
-      <material>
-        <ambient>0.8 0 0 1</ambient>
-        <diffuse>0.8 0 0 1</diffuse>
-        <specular>0.8 0 0 1</specular>
-      </material>
-    </visual>
-  </gazebo>
-  <gazebo reference="base_link">
-    <visual>
-      <material>
-        <ambient>1 1 1 1</ambient>
-        <diffuse>1 1 1 1</diffuse>
-        <specular>1 1 1 1</specular>
-      </material>
-    </visual>
-  </gazebo>
-  <gazebo reference="base_scan">
-    <visual>
-      <material>
-        <ambient>0 0 0 1</ambient>
-        <diffuse>0 0 0 1</diffuse>
-        <specular>0 0 0 1</specular>
-      </material>
-    </visual>
   </gazebo>
 </robot>
